File: orkman.kicad_pcb (KiCad board)
At the start: 2 copper layers, 29.2 x 42.1 mm, 25 parts, among them J1 Stomp_Connector, J2 Power_Connector, U1 TL072

Commit message: updated to KiCad 6.0
Other:
- net class Default removed
